Commit message: Change URDF

File: examples/indy7/indy7_dualArm.urdf (robot description, URDF)
Before this commit: robot IndyDualArm, 18 links, 17 joints
Links:
- link l_1: geometry collision mesh filename=meshes/collision/Indy7_1.stl; visual mesh filename=meshes/collision/Indy7_1.stl
- link l_2: geometry collision mesh filename=meshes/collision/Indy7_2.stl; visual mesh filename=meshes/collision/Indy7_2.stl
- link l_3: geometry collision mesh filename=meshes/collision/Indy7_3.stl; visual mesh filename=meshes/collision/Indy7_3.stl
- link l_4: geometry collision mesh filename=meshes/collision/Indy7_4.stl; visual mesh filename=meshes/collision/Indy7_4.stl
- link l_5: geometry collision mesh filename=meshes/collision/Indy7_5.stl; visual mesh filename=meshes/collision/Indy7_5.stl
- link l_6: geometry collision mesh filename=meshes/collision/Indy7_6.stl; visual mesh filename=meshes/collision/Indy7_6.stl
- link r_1: geometry collision mesh filename=meshes/collision/Indy7_1.stl; visual mesh filename=meshes/collision/Indy7_1.stl
- link r_2: geometry collision mesh filename=meshes/collision/Indy7_2.stl; visual mesh filename=meshes/collision/Indy7_2.stl
- link r_3: geometry collision mesh filename=meshes/collision/Indy7_3.stl; visual mesh filename=meshes/collision/Indy7_3.stl
- link r_4: geometry collision mesh filename=meshes/collision/Indy7_4.stl; visual mesh filename=meshes/collision/Indy7_4.stl
- link r_5: geometry collision mesh filename=meshes/collision/Indy7_5.stl; visual mesh filename=meshes/collision/Indy7_5.stl
- link r_6: geometry collision mesh filename=meshes/collision/Indy7_6.stl; visual mesh filename=meshes/collision/Indy7_6.stl
Joints:
- joint l_body_fixed: origin xyz=0 0.1551 1.2924 rpy= 2.091 0 3.141592 -> xyz=0 0.1551 1.2924 rpy=-2.091 0 0
- joint world_fixed: origin xyz=0 0 0 rpy=0 0 3.141592 -> xyz=0 0 0 rpy=0 0 0

File: slx/indy7/indy7_dualArm.urdf (robot description, URDF)
Before this commit: robot IndyDualArm, 18 links, 17 joints
Joints:
- joint l_body_fixed: origin xyz=0 0.1551 1.2924 rpy= 2.091 0 3.141592 -> xyz=0 0.1551 1.2924 rpy=-2.091 0 0

Commit message: Chage URDF_

File: examples/indy7/indy7_dualArm.urdf (robot description, URDF)
Before this commit: robot IndyDualArm, 18 links, 17 joints
Links:
- link l_0: mass 1.59306955 -> 1.6703078
- link l_1: mass 11.8030102 -> 11.44444535; geometry collision mesh filename=meshes/collision/Indy7_1.stl; visual mesh filename=meshes/visual/Indy7_1.stl
- link l_2: mass 7.99292141 -> 5.84766553; geometry collision mesh filename=meshes/collision/Indy7_2.stl; visual mesh filename=meshes/visual/Indy7_2.stl
- link l_3: mass 2.99134127 -> 2.68206064; geometry collision mesh filename=meshes/collision/Indy7_3.stl; visual mesh filename=meshes/visual/Indy7_3.stl
- link l_4: mass 2.12317035 -> 2.12987371; geometry collision mesh filename=meshes/collision/Indy7_4.stl; visual mesh filename=meshes/visual/Indy7_4.stl
- link l_5: mass 2.28865091 -> 2.22412271; geometry collision mesh filename=meshes/collision/Indy7_5.stl; visual mesh filename=meshes/visual/Indy7_5.stl
- link l_6: mass 0.40083918 -> 0.38254932; geometry collision mesh filename=meshes/collision/Indy7_6.stl; visual mesh filename=meshes/visual/Indy7_6.stl
- link r_0: mass 1.59306955 -> 1.6703078
- link r_1: mass 11.8030102 -> 11.44444535; geometry collision mesh filename=meshes/collision/Indy7_1.stl; visual mesh filename=meshes/visual/Indy7_1.stl
- link r_2: mass 7.99292141 -> 5.84766553; geometry collision mesh filename=meshes/collision/Indy7_2.stl; visual mesh filename=meshes/visual/Indy7_2.stl
- link r_3: mass 2.99134127 -> 2.68206064; geometry collision mesh filename=meshes/collision/Indy7_3.stl; visual mesh filename=meshes/visual/Indy7_3.stl
- link r_4: mass 2.12317035 -> 2.12987371; geometry collision mesh filename=meshes/collision/Indy7_4.stl; visual mesh filename=meshes/visual/Indy7_4.stl
- link r_5: mass 2.28865091 -> 2.22412271; geometry collision mesh filename=meshes/collision/Indy7_5.stl; visual mesh filename=meshes/visual/Indy7_5.stl
- link r_6: mass 0.40083918 -> 0.38254932; geometry collision mesh filename=meshes/collision/Indy7_6.stl; visual mesh filename=meshes/visual/Indy7_6.stl
Joints:
- joint l_joint_0: limit lower=-3.054325556 upper=3.054325556 effort=10 velocity=1 -> lower=-3.05432619099 upper=3.05432619099 effort=431.97 velocity=2.61799333; origin xyz=0 0 0.08 rpy=0 0 0 -> xyz=0 0 0.0775 rpy=0 0 0
- joint l_joint_1: limit lower=-3.054325556 upper=3.054325556 effort=10 velocity=1 -> lower=-3.05432619099 upper=3.05432619099 effort=431.97 velocity=2.61799388; origin xyz=0 -0.109 0.222 rpy=1.5707 1.5707 0 -> xyz=0 -0.109 0.222 rpy=1.570796327 1.570796327 0
- joint l_joint_2: limit lower=-3.054325556 upper=3.054325556 effort=10 velocity=1 -> lower=-3.05432619099 upper=3.05432619099 effort=197.23 velocity=2.61799388
- joint l_joint_3: limit lower=-3.054325556 upper=3.054325556 effort=10 velocity=1 -> lower=-3.05432619099 upper=3.05432619099 effort=79.79 velocity=3.14159265; origin xyz=-0.267 0 -0.075 rpy=-1.5707 0 1.5707 -> xyz=-0.267 0 -0.075 rpy=-1.570796327 0 1.570796327
- joint l_joint_4: limit lower=-3.054325556 upper=3.054325556 effort=10 velocity=1 -> lower=-3.05432619099 upper=3.05432619099 effort=79.79 velocity=3.14159265; origin xyz=0 -0.114 0.083 rpy=1.5707 1.5707 0 -> xyz=0 -0.114 0.083 rpy=1.570796327 1.570796327 0
- joint l_joint_5: limit lower=-3.752457111 upper=3.752457111 effort=10 velocity=1 -> lower=-3.75245789179 upper=3.75245789179 effort=79.79 velocity=3.14159265; origin xyz=-0.168 0 0.069 rpy=-1.5707 0 1.5707 -> xyz=-0.168 0 0.069 rpy=-1.570796327 0 1.570796327
- joint r_joint_0: limit lower=-3.054325556 upper=3.054325556 effort=10 velocity=1 -> lower=-3.05432619099 upper=3.05432619099 effort=431.97 velocity=2.61799333
- joint r_joint_1: limit lower=-3.054325556 upper=3.054325556 effort=10 velocity=1 -> lower=-3.05432619099 upper=3.05432619099 effort=431.97 velocity=2.61799388; origin xyz=0 -0.109 0.222 rpy=1.5707 1.5707 0 -> xyz=0 -0.109 0.222 rpy=1.570796327 1.570796327 0
- joint r_joint_2: limit lower=-3.054325556 upper=3.054325556 effort=10 velocity=1 -> lower=-3.05432619099 upper=3.05432619099 effort=197.23 velocity=2.61799388
- joint r_joint_3: limit lower=-3.054325556 upper=3.054325556 effort=10 velocity=1 -> lower=-3.05432619099 upper=3.05432619099 effort=79.79 velocity=3.14159265; origin xyz=-0.267 0 -0.075 rpy=-1.5707 0 1.5707 -> xyz=-0.267 0 -0.075 rpy=-1.570796327 0 1.570796327
- joint r_joint_4: limit lower=-3.054325556 upper=3.054325556 effort=10 velocity=1 -> lower=-3.05432619099 upper=3.05432619099 effort=79.79 velocity=3.14159265; origin xyz=0 -0.114 0.083 rpy=1.5707 1.5707 0 -> xyz=0 -0.114 0.083 rpy=1.570796327 1.570796327 0
- joint r_joint_5: limit lower=-3.752457111 upper=3.752457111 effort=10 velocity=1 -> lower=-3.75245789179 upper=3.75245789179 effort=79.79 velocity=3.14159265; origin xyz=-0.168 0 0.069 rpy=-1.5707 0 1.5707 -> xyz=-0.168 0 0.069 rpy=-1.570796327 0 1.570796327

Commit message: Add

File: examples/indy7/indy7_dualArm.urdf (robot description, URDF)
Before this commit: robot IndyDualArm, 18 links, 17 joints
Joints:
- joint l_body_fixed: origin xyz=0 0.1551 1.2924 rpy=-2.091 0 0 -> xyz=0 0.1551 0.61651 rpy=-2.091 0 0
- joint r_body_fixed: origin xyz=0 -0.1551 1.2924 rpy= 2.091 0 0 -> xyz=0 -0.1551 0.61651 rpy= 2.091 0 0

File: examples/indy7/indy7_dualArm_vis.urdf (robot description, URDF)
Before this commit: robot IndyDualArm, 18 links, 17 joints
Joints:
- joint l_body_fixed: origin xyz=0 0.1551 1.2924 rpy=-2.091 0 0 -> xyz=0 0.1551 0.61651 rpy=-2.091 0 0
- joint r_body_fixed: origin xyz=0 -0.1551 1.2924 rpy= 2.091 0 0 -> xyz=0 -0.1551 0.61651 rpy= 2.091 0 0
